File: ledBloom.brd (EAGLE design)
At the start: 11.4 x 14.6 mm, 4 parts, among them J1 455-1750-1-ND, J2 455-1750-1-ND, U1 WS2812

Commit message: adding production files
Parts:
- removed U1: WS2812, SparkFun-LED:LED-TRICOLOR-5050-IC
- added D1: WS2812B, SparkFun-LED:WS2812B
- moved J1 10.8 mm to (5.71, 2.54)
- moved C1 10.8 mm to (3.65, 8.10)
- moved J2 10.7 mm to (10.8, 13.3)
Connections:
- net DI: now also D1.4; no longer U1.2
- net DO: now also D1.2; no longer U1.1
- net GND: now also D1.3; no longer U1.6
- net VCC: now also D1.1; no longer U1.3, U1.5
Routing:
- net GND: track 25.2 -> 0.00 mm, vias 3 -> 2
- net VCC: track 22.8 -> 18.9 mm
- net DO: track 7.00 -> 9.72 mm

Commit message: Updating Silk, adding Desert Bloom to Sch
Other:
- board text added: "Desert Bloom Addressable LED"
- board text removed: "Desert Bloom Addressable RGB LED"
Changed lines of the file:
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@@
 <text x="11.58875" y="11.90625" size="0.8128" layer="21" font="vector" ratio="15" rot="R180">DO</text>
 <text x="10.00125" y="11.90625" size="0.8128" layer="22" font="vector" ratio="15" rot="MR180">DO</text>
-<text x="11.27125" y="4.1275" size="0.8128" layer="22" font="vector" ratio="15" rot="MR0">DI</text>
-<text x="9.36625" y="4.1275" size="0.8128" layer="22" font="vector" ratio="15" rot="MR0">GND</text>
+<text x="11.43" y="4.1275" size="0.8128" layer="22" font="vector" ratio="15" rot="MR0">DI</text>
+<text x="9.2075" y="4.1275" size="0.8128" layer="22" font="vector" ratio="15" rot="MR0">GND</text>
 <text x="6.35" y="4.1275" size="0.8128" layer="22" font="vector" ratio="15" rot="MR0">5V</text>
-<text x="8.09625" y="8.41375" size="0.8128" layer="22" font="vector" ratio="20" rot="SMR0" align="center">Desert Bloom
+<text x="8.255" y="8.255" size="0.8128" layer="22" font="vector" ratio="20" rot="SMR0" align="center">Desert Bloom
 Addressable
-RGB LED</text>
+LED</text>
 </plain>
 <attributes>
